File: kicad/transmitter-rev-a/transmitter-rev-a.kicad_pcb (KiCad board)
At the start: 2 copper layers, 36 parts, among them J13 GPIO, J14 GPIO, J2 RGB LED, J3 GPIO, J4 Battery, J5 Debug UART, J8 GPIO, Q1 Q_PMOS_GSD, SW1 SW_SPST, SW2 SW_SPST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

Commit message: Transmitter PCB progress
Parts:
- removed U4: AMS1117-3.3, Package_TO_SOT_SMD:SOT-223-3_TabPin2
- added C1: 10u, Capacitor_SMD:C_0603_1608Metric, F.Cu at (124.9, 112.7)
- added J1: USB C, easyeda2kicad:USB-SMD_GT-USB-7010AN, F.Cu at (124.1, 135.4)
- added J15: VSYS_VOLTAGE, Connector_PinHeader_2.54mm:PinHeader_1x02_P2.54mm_Vertical, F.Cu at (130.4, 126.8)
- added J6: VSYS_VOLTAGE, Connector_PinHeader_2.54mm:PinHeader_1x02_P2.54mm_Vertical, F.Cu at (121.1, 126.8)
- added J7: VSYS_VOLTAGE, Connector_PinHeader_2.54mm:PinHeader_1x02_P2.54mm_Vertical, F.Cu at (125.7, 126.8)
- added J9: 1.8 TFT, Connector_PinSocket_2.54mm:PinSocket_1x08_P2.54mm_Vertical, F.Cu at (99.0, 107.3)
- added SW3: SWITCH 1, Custom3:On-Off-On_Switch, F.Cu at (105.6, 125.2)
- added SW4: SWITCH 2, Custom3:On-Off-On_Switch, F.Cu at (114.4, 125.2)
- added U7: WL2803K33-5/TR, easyeda2kicad:SOT-89-5_L4.5-W2.5-P1.50-LS4.5-TL, F.Cu at (125.8, 108.0)
- J2: value RGB LED -> VSYS_VOLTAGE; footprint Connector_PinSocket_2.54mm:PinSocket_1x03_P2.54mm_Vertical -> Connector_PinHeader_2.54mm:PinHeader_1x02_P2.54mm_Vertical
- U1: value COM-09032 -> Joystick Left; footprint Custom:COM-09032 -> Custom3:PS4tJoystick
- moved U1 74.7 mm to (208.3, 93.8)
Connections:
- C8 pad 1: BATT_1_PLUS -> VBAT
- J2 pad 1: RGB_LED -> +5V
- J2 pad 2: +5V -> GND
- U2 pad 5: BATT_1_PLUS -> VBAT
Routing:
- net unconnected-(U1-V--PadV3): track 15.1 -> 0.00 mm

Commit message: Transmitter pcb progress. Schematic mostly done
Parts:
- removed J13, J14, J3, J8: GPIO, Connector_PinSocket_2.54mm:PinSocket_1x04_P2.54mm_Vertical
- removed J7: VSYS_VOLTAGE, Connector_PinHeader_2.54mm:PinHeader_1x02_P2.54mm_Vertical
- added C2: 10u, Capacitor_SMD:C_0603_1608Metric, B.Cu at (174.1, 85.9)
- added D2: D_Schottky, Diode_SMD:D_SOD-323, B.Cu at (142.8, 100.0)
- added J10: OLED, Connector_PinSocket_2.54mm:PinSocket_1x04_P2.54mm_Vertical, F.Cu at (154.2, 76.2)
- added J11: Vib Motor, Custom3:Conn_01x02_no_Silk, F.Cu at (145.1, 102.2)
- added J12: Audio Player, Connector_PinSocket_2.54mm:PinSocket_1x07_P2.54mm_Vertical, F.Cu at (171.5, 100.4)
- added Q4: Q_NMOS_Depletion_GSD, Package_TO_SOT_SMD:SOT-23, B.Cu at (142.8, 96.8)
- added R10: 1k, Resistor_SMD:R_0402_1005Metric, B.Cu at (160.3, 101.5)
- added R11: 10k, Resistor_SMD:R_0402_1005Metric, B.Cu at (142.7, 94.3)
- added R12: 1k, Resistor_SMD:R_0402_1005Metric, B.Cu at (142.7, 93.2)
- added R15: 47k, Resistor_SMD:R_0402_1005Metric, F.Cu at (173.4, 78.5)
- added R16: 47k, Resistor_SMD:R_0402_1005Metric, F.Cu at (140.2, 78.5)
- added R17: 10k, Resistor_SMD:R_0402_1005Metric, F.Cu at (137.6, 78.5)
- added R18: 33k, Resistor_SMD:R_0402_1005Metric, F.Cu at (134.9, 78.5)
- added R19: 33k, Resistor_SMD:R_0402_1005Metric, F.Cu at (178.7, 78.5)
- added R20: 10k, Resistor_SMD:R_0402_1005Metric, F.Cu at (176.1, 78.5)
- added R21: 10k, Resistor_SMD:R_0402_1005Metric, F.Cu at (175.8, 102.8)
- added R22: 10k, Resistor_SMD:R_0402_1005Metric, B.Cu at (123.0, 98.3)
- added SW5: Battery, Custom3:SideSwitch_5_Legs, F.Cu at (146.9, 111.7)
- added U4: Joystick left, Custom3:PS4tJoystick, F.Cu at (120.6, 113.6)
- C3, C6, C7, C8, D1, Q1, R2, R3, R4, R5, R6, R8, R9, U2: moved to B.Cu
- J15, J2, J6: footprint Connector_PinHeader_2.54mm:PinHeader_1x02_P2.54mm_Vertical -> Custom3:Conn_01x02_no_Silk
- U1: value Joystick Left -> Joystick right
- U7: footprint easyeda2kicad:SOT-89-5_L4.5-W2.5-P1.50-LS4.5-TL -> Package_TO_SOT_SMD:SOT-89-5; moved to B.Cu
- moved SW4 75.7 mm to (169.6, 73.5), turned to 90 degrees
- moved J6 71.7 mm to (178.7, 84.2)
- moved J15 66.5 mm to (181.5, 84.2)
- moved SW3 64.2 mm to (143.7, 73.5), turned to -90 degrees
- moved D3 52.9 mm to (188.4, 84.7), turned to 180 degrees
- moved D4 52.1 mm to (188.4, 88.3), turned to 180 degrees
- moved R14 43.4 mm to (168.6, 87.7)
- moved J1 43.1 mm to (158.5, 109.5)
- moved U6 42.7 mm to (154.3, 70.6), turned to 90 degrees
- moved R13 42.7 mm to (168.6, 86.4)
- moved C15 40.8 mm to (151.6, 72.0), turned to -90 degrees
- moved J2 39.0 mm to (176.4, 84.2)
- moved C5 37.9 mm to (146.0, 85.0), turned to 180 degrees
- moved C4 37.7 mm to (146.0, 86.4), turned to 180 degrees
- moved C8 36.7 mm to (157.3, 92.3)
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Connections:
- J2 pad 1: +5V -> VSYS
- J4 pad 1: VBAT -> Net-(J4-Pin_1)
- U1 pad 1: (no net) -> +3.3V
- U1 pad 2: (no net) -> JOYSTICK_RIGHT_HORI
- U1 pad 3: (no net) -> GND
- U1 pad 4: (no net) -> GND
- U1 pad 5: (no net) -> JOYSTICK_RIGHT_VERT
- U1 pad 6: (no net) -> +3.3V
- U1 pad 7: (no net) -> JOYSTICK_RIGHT_BTN
- U1 pad 8: (no net) -> Net-(U1-BFL)
- U3 pad 10: unconnected-(U3-GPIO17/U1TXD/ADC2_CH6-Pad10) -> JOYSTICK_LEFT_BTN
- U3 pad 11: unconnected-(U3-GPIO18/U1RXD/ADC2_CH7/CLK_OUT3-Pad11) -> JOYSTICK_LEFT_VERT
- U3 pad 12: unconnected-(U3-GPIO8/TOUCH8/ADC1_CH7/SUBSPICS1-Pad12) -> JOYSTICK_LEFT_HORI
- U3 pad 22: unconnected-(U3-GPIO14/TOUCH14/ADC2_CH3/FSPIWP/FSPIDQS/SUBSPIWP-Pad22) -> JOYSTICK_RIGHT_HORI
- U3 pad 23: unconnected-(U3-GPIO21-Pad23) -> JOYSTICK_RIGHT_VERT
- U3 pad 24: unconnected-(U3-GPIO47/SPICLK_P/SUBSPICLK_P_DIFF-Pad24) -> JOYSTICK_RIGHT_BTN
- U3 pad 28: unconnected-(U3-SPIIO6/GPIO35/FSPID/SUBSPID-Pad28) -> AUDIO_LRC
- U3 pad 29: unconnected-(U3-SPIIO7/GPIO36/FSPICLK/SUBSPICLK-Pad29) -> AUDIO_BCLK
- U3 pad 30: unconnected-(U3-SPIDQS/GPIO37/FSPIQ/SUBSPIQ-Pad30) -> AUDIO_DIN
- U3 pad 38: unconnected-(U3-GPIO2/TOUCH2/ADC1_CH1-Pad38) -> LED_RED
- U3 pad 39: unconnected-(U3-GPIO1/TOUCH1/ADC1_CH0-Pad39) -> LED_BLUE
- U6 pad 1: GND -> +3.3V
- U6 pad 2: +3.3V -> GND
- U6 pad 3: NRF_CE -> NRF_CSN
- U6 pad 4: NRF_CSN -> NRF_CE
- U6 pad 5: NRF_SCK -> NRF_MOSI
- U6 pad 6: NRF_MOSI -> NRF_SCK
- U6 pad 7: NRF_MISO -> NRF_IRQ
- U6 pad 8: NRF_IRQ -> NRF_MISO
- U7 pad 2: GND -> unconnected-(U7-GND-Pad2)
Routing:
- net +3.3V: track 0.00 -> 214.2 mm, vias 0 -> 3
- net VSYS: track 0.00 -> 72.6 mm, vias 0 -> 2
- net JOYSTICK_LEFT_BTN: track 0.00 -> 60.0 mm
- net VBAT: track 0.00 -> 49.8 mm
- net ~{NRESET}: track 0.00 -> 38.2 mm, vias 0 -> 2
- net JOYSTICK_RIGHT_HORI: track 0.00 -> 37.6 mm
- net JOYSTICK_RIGHT_BTN: track 0.00 -> 36.1 mm
- net VBUS: track 0.00 -> 34.3 mm, vias 0 -> 2
- net JOYSTICK_LEFT_HORI: track 0.00 -> 34.1 mm
- net NRF_CSN: track 0.00 -> 31.6 mm
- net NRF_SCK: track 0.00 -> 30.2 mm
- net NRF_CE: track 0.00 -> 29.1 mm
- net NRF_IRQ: track 0.00 -> 28.5 mm, vias 0 -> 2
- net TX0: track 0.00 -> 27.5 mm, vias 0 -> 1
- net NRF_MOSI: track 0.00 -> 27.4 mm, vias 0 -> 2
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- added copper zone on B.Cu, net GND
- added copper zone on F.Cu, net GND
Other:
- board outline added: 94.2 x 64.6 mm

Commit message: Transmitter PCB almost done in kicad
Parts:
- removed J10: OLED, Connector_PinSocket_2.54mm:PinSocket_1x04_P2.54mm_Vertical
- added H1: MountingHole_Pad, MountingHole:MountingHole_3.2mm_M3_Pad_Via, F.Cu at (138.0, 73.0)
- added H2: MountingHole_Pad, MountingHole:MountingHole_3.2mm_M3_Pad_Via, F.Cu at (176.0, 73.0)
- added H3: MountingHole_Pad, MountingHole:MountingHole_3.2mm_M3_Pad_Via, F.Cu at (119.3, 127.0)
- added H4: MountingHole_Pad, MountingHole:MountingHole_3.2mm_M3_Pad_Via, F.Cu at (195.0, 127.0)
- added R23: 10k, Resistor_SMD:R_0402_1005Metric, B.Cu at (127.2, 95.7)
- added R24: 10k, Resistor_SMD:R_0402_1005Metric, B.Cu at (134.9, 102.5)
- added R25: 10k, Resistor_SMD:R_0402_1005Metric, B.Cu at (181.5, 108.2)
- added SW6: KAN0641-0431B-L, easyeda2kicad:KEY-SMD_4P-L6.0-W6.0-P4.50-LS10.0, F.Cu at (135.3, 107.6)
- added SW7: KAN0641-0431B-L, easyeda2kicad:KEY-SMD_4P-L6.0-W6.0-P4.50-LS10.0, F.Cu at (177.2, 107.6)
- C1, C15, J4, R15, R16, R17, R18, R19, R20, R21: moved to B.Cu
- moved D3 68.9 mm to (120.8, 97.6), turned to 0 degrees
- moved R13 28.3 mm to (146.6, 104.2), turned to 180 degrees
- moved SW4 22.0 mm to (190.6, 80.3), turned to 0 degrees
- moved SW3 20.8 mm to (124.0, 80.3), turned to 0 degrees
- moved R9 19.4 mm to (157.9, 90.5), turned to -90 degrees
- moved R6 18.8 mm to (159.2, 90.5), turned to -90 degrees
- moved R5 18.3 mm to (160.5, 90.5), turned to 90 degrees
- moved R21 17.9 mm to (193.6, 100.4), turned to 90 degrees
- moved R8 17.4 mm to (156.4, 90.5), turned to 90 degrees
- moved R15 14.7 mm to (187.2, 83.6), turned to -90 degrees
- moved R19 14.1 mm to (187.1, 89.8), turned to 90 degrees
- moved R20 13.8 mm to (187.2, 86.7), turned to 90 degrees
- moved R16 13.5 mm to (127.6, 83.4), turned to -90 degrees
- moved R18 13.3 mm to (127.6, 89.6), turned to 90 degrees
- moved J12 13.1 mm to (183.4, 105.8)
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Connections:
- J9 pad 1: DISPLAY_TFT_LED -> Net-(J9-Pin_1)
- U3 pad 10: JOYSTICK_LEFT_BTN -> DISPLAY_TFT_SDA
- U3 pad 11: JOYSTICK_LEFT_VERT -> DISPLAY_TFT_SCK
- U3 pad 12: JOYSTICK_LEFT_HORI -> AUX_SWITCH_1
- U3 pad 15: unconnected-(U3-GPIO3/TOUCH3/ADC1_CH2-Pad15) -> JOYSTICK_LEFT_BTN
- U3 pad 16: unconnected-(U3-GPIO46-Pad16) -> LED_BLUE
- U3 pad 17: unconnected-(U3-GPIO9/TOUCH9/ADC1_CH8/FSPIHD/SUBSPIHD-Pad17) -> JOYSTICK_LEFT_VERT
- U3 pad 18: unconnected-(U3-GPIO10/TOUCH10/ADC1_CH9/FSPICS0/FSPIIO4/SUBSPICS0-Pad18) -> JOYSTICK_LEFT_HORI
- U3 pad 19: unconnected-(U3-GPIO11/TOUCH11/ADC2_CH0/FSPID/FSPIIO5/SUBSPID-Pad19) -> JOYSTICK_RIGHT_HORI
- U3 pad 20: unconnected-(U3-GPIO12/TOUCH12/ADC2_CH1/FSPICLK/FSPIIO6/SUBSPICLK-Pad20) -> JOYSTICK_RIGHT_VERT
- U3 pad 21: unconnected-(U3-GPIO13/TOUCH13/ADC2_CH2/FSPIQ/FSPIIO7/SUBSPIQ-Pad21) -> JOYSTICK_RIGHT_BTN
- U3 pad 22: JOYSTICK_RIGHT_HORI -> BATT_VOLTAGE
- U3 pad 23: JOYSTICK_RIGHT_VERT -> ~{CHRG}
- U3 pad 24: JOYSTICK_RIGHT_BTN -> USB_SENSE
- U3 pad 25: unconnected-(U3-GPIO48/SPICLK_N/SUBSPICLK_N_DIFF-Pad25) -> VIBRATION_MOTOR
- U3 pad 31: unconnected-(U3-GPIO38/FSPIWP/SUBSPIWP-Pad31) -> BTN_RIGHT
- U3 pad 32: unconnected-(U3-MTCK/GPIO39/CLK_OUT3/SUBSPICS1-Pad32) -> BTN_LEFT
- U3 pad 33: unconnected-(U3-MTDO/GPIO40/CLK_OUT2-Pad33) -> NRF_IRQ
- U3 pad 34: unconnected-(U3-MTDI/GPIO41/CLK_OUT1-Pad34) -> NRF_MOSI
- U3 pad 35: unconnected-(U3-MTMS/GPIO42-Pad35) -> NRF_MISO
- U3 pad 39: LED_BLUE -> AUX_SWITCH_2
- U3 pad 4: unconnected-(U3-GPIO4/TOUCH4/ADC1_CH3-Pad4) -> NRF_SCK
- U3 pad 5: unconnected-(U3-GPIO5/TOUCH5/ADC1_CH4-Pad5) -> NRF_CE
- U3 pad 6: unconnected-(U3-GPIO6/TOUCH6/ADC1_CH5-Pad6) -> NRF_CSN
- U3 pad 7: unconnected-(U3-GPIO7/TOUCH7/ADC1_CH6-Pad7) -> DISPLAY_TFT_CS
- U3 pad 8: unconnected-(U3-GPIO15/U0RTS/ADC2_CH4/XTAL_32K_P-Pad8) -> DISPLAY_TFT_RESET
- U3 pad 9: unconnected-(U3-GPIO16/U0CTS/ADC2_CH5/XTAL_32K_N-Pad9) -> DISPLAY_TFT_A0
Routing:
- net BTN_LEFT: track 0.00 -> 47.7 mm, vias 0 -> 2
- net JOYSTICK_LEFT_VERT: track 0.00 -> 45.3 mm
- net +3.3V: track 214.2 -> 258.1 mm, vias 3 -> 6
- net VIBRATION_MOTOR: track 0.00 -> 37.2 mm, vias 0 -> 1
- net GND: track 8.38 -> 44.7 mm, vias 2 -> 68
- net AUX_SWITCH_1: track 7.03 -> 33.2 mm
- net JOYSTICK_LEFT_BTN: track 60.0 -> 34.6 mm
- net BTN_RIGHT: track 0.00 -> 24.6 mm, vias 0 -> 2
- net AUX_SWITCH_2: track 4.75 -> 28.4 mm, vias 0 -> 1
- net BATT_VOLTAGE: track 0.00 -> 20.8 mm, vias 0 -> 1
- net USB_SENSE: track 0.00 -> 20.1 mm, vias 0 -> 1
- net DISPLAY_TFT_LED: track 18.5 -> 0.00 mm
- net ~{CHRG}: track 0.00 -> 16.0 mm, vias 0 -> 1
- net AUDIO_LRC: track 5.22 -> 20.2 mm
- net Net-(D4-A): track 19.5 -> 33.8 mm
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Other:
- outline, holes or cut-outs redrawn
- board text added: "+"
- board text added: "-"
- board text added: "3V3"
- board text added: "A0"
- board text added: "BCLK"
- board text added: "BOOT"
- board text added: "CS"
- board text added: "DIN"
- board text added: "ESP32-S3"
- board text added: "GND"
- board text added: "LRC"
- board text added: "RESET"
- board text added: "RST"
- board text added: "RX0"
- board text added: "SCK"
- board text added: "SDA"
- board text added: "TX0"
- board text added: "VBAT (1s)"
- board text added: "VSYS"
- board text added: "Vib Motor"

Commit message: Ordered PCBs for rev A
Routing:
- net VSYS: track 76.6 -> 77.7 mm
- net USB-: track 30.1 -> 29.1 mm
- net BTN_LEFT: track 47.7 -> 47.0 mm
- net NRF_MISO: track 24.2 -> 24.7 mm
- net GND: vias 68 -> 70
- net (no net): vias 2 -> 0
Other:
- outline, holes or cut-outs redrawn
- board text added: "rev. A"
