File: kicad/transmitter-rev-a/transmitter-rev-a.kicad_sch (KiCad schematic)
At the start: 45 parts, among them J1 USB C, J13 GPIO, J14 GPIO, J2 RGB LED, J3 GPIO, J4 Battery, J5 Debug UART, J6 VSYS_VOLTAGE, J7 VSYS_VOLTAGE, J8 GPIO, Q1 Q_PMOS_GSD, SW1 SW_SPST, SW2 SW_SPST, U1 Joystick Left, U2 TP4056, U3 ESP32-S3-WROOM-1, U5 Joystick Right, U6 NRF24L01, U7 WL2803K33-5/TR

Commit message: Transmitter PCB progress
Parts:
- removed J2: RGB LED, Connector_PinSocket_2.54mm:PinSocket_1x03_P2.54mm_Vertical, symbol Connector_Generic:Conn_01x03
- removed U1: Joystick Left, Custom:COM-09032, symbol Custom:COM-09032
- removed U5: Joystick Right, Custom:COM-09032, symbol Custom:COM-09032
- added C1: 10u, Capacitor_SMD:C_0603_1608Metric, symbol Device:C_Small
- added D2: D_Schottky, symbol Device:D_Schottky
- added J10: OLED, symbol Connector_Generic:Conn_01x04
- added J11: Vib Motor, symbol Connector_Generic:Conn_01x02
- added J12: Audio Player, symbol Connector_Generic:Conn_01x07
- added J15, J2: VSYS_VOLTAGE, Connector_PinHeader_2.54mm:PinHeader_1x02_P2.54mm_Vertical, symbol Connector_Generic:Conn_01x02
- added J9: 1.8 TFT, Connector_PinSocket_2.54mm:PinSocket_1x08_P2.54mm_Vertical, symbol Connector_Generic:Conn_01x08
- added Q2: NMOS, symbol Simulation_SPICE:NMOS
- added R11, R17, R20, R21, R22: 10k, symbol Device:R_Small
- added R12: 1k, symbol Device:R_Small
- added R15, R16: 47k, symbol Device:R_Small
- added R18, R19: 33k, symbol Device:R_Small
- added SW3: SWITCH 1, Custom3:On-Off-On_Switch, symbol Switch:SW_DPDT_x2
- added SW4: SWITCH 2, Custom3:On-Off-On_Switch, symbol Switch:SW_DPDT_x2
- added U1: Joystick right, Custom3:PS4tJoystick, symbol custom3:PS4Joystick
- added U4: Joystick left, Custom3:PS4tJoystick, symbol custom3:PS4Joystick
Connections:
- net +3.3V: now also C1.1, J10.2 (Pin_2), J12.7 (Pin_7), J15.1 (Pin_1), J9.8 (Pin_8), SW3.2 (B), SW4.2 (B), U1.1 (H+), U1.6 (V+), U4.1 (H+), U4.6 (V+)
- net +5V: now also J2.1 (Pin_1)
- net GND: now also C1.2, J10.1 (Pin_1), J12.6 (Pin_6), J15.2 (Pin_2), J2.2 (Pin_2), J9.7 (Pin_7), Q2.3 (S), R11.2, R17.2, R20.2, R21.2, R22.2, U1.3 (H-), U1.4 (V-), U4.3 (H-), U4.4 (V-)
- net JOYSTICK_LEFT_BTN: now also U4.7 (BBR)
- net JOYSTICK_LEFT_HORI: now also U4.2 (H)
- net JOYSTICK_LEFT_VERT: now also U4.5 (V)
- net JOYSTICK_RIGHT_BTN: now also U1.7 (BBR)
- net JOYSTICK_RIGHT_HORI: now also U1.2 (H)
- net JOYSTICK_RIGHT_VERT: now also U1.5 (V)
- net VSYS: now also D2.1 (K), J11.1 (Pin_1)
- new net: R22.1, U4.8 (BFR)
- new net: R15.1, SW4.1 (A)
- new net: Q2.2 (G), R11.1, R12.2
- new net: D2.2 (A), J11.2 (Pin_2), Q2.1 (D)
- new net: R21.1, U1.8 (BFR)
- new net: R19.1, SW4.3 (C)
- new net: R18.1, SW3.3 (C)
- new net: R16.1, SW3.1 (A)
- new net AUX_SWITCH_1: R16.2, R17.1, R18.2
- new net AUX_SWITCH_2: R15.2, R19.2, R20.1
- new net BCLK: J12.2 (Pin_2)
- new net DIN: J12.3 (Pin_3)
- new net DISPLAY_OLED_SCL: J10.3 (Pin_3)
- new net DISPLAY_OLED_SDA: J10.4 (Pin_4)
- new net DISPLAY_TFT_A0: J9.4 (Pin_4)
- new net DISPLAY_TFT_CS: J9.6 (Pin_6)
- new net DISPLAY_TFT_LED: J9.1 (Pin_1)
- new net DISPLAY_TFT_RESET: J9.5 (Pin_5)
- new net DISPLAY_TFT_SCK: J9.2 (Pin_2)
- new net DISPLAY_TFT_SDA: J9.3 (Pin_3)
- new net GAIN: J12.4 (Pin_4)
- new net LRC: J12.1 (Pin_1)
- new net SD: J12.5 (Pin_5)
- new net VIBRATION_MOTOR: R12.1
- no-connect marks 5 -> 3
Other:
- note added: "Audio"
- note added: "Buttons & Switches"
- note added: "Displays"
- note added: "Joysticks"
- note added: "Vibration motor"
- note removed: "Buttons"
- moved on the sheet: C7, C8, D3, D4, J13, J14, J3, J8, R10, R13, R14, SW1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

Commit message: Transmitter pcb progress. Schematic mostly done
Parts:
- removed J13, J14, J3, J8: GPIO, Connector_PinSocket_2.54mm:PinSocket_1x04_P2.54mm_Vertical, symbol Connector_Generic:Conn_01x04
- removed J7: VSYS_VOLTAGE, Connector_PinHeader_2.54mm:PinHeader_1x02_P2.54mm_Vertical, symbol Connector_Generic:Conn_01x02
- removed Q2: NMOS, symbol Simulation_SPICE:NMOS
- added C2: 10u, Capacitor_SMD:C_0603_1608Metric, symbol Device:C_Small
- added Q4: Q_NMOS_Depletion_GSD, Package_TO_SOT_SMD:SOT-23, symbol Device:Q_NMOS_Depletion_GSD
- added SW5: Battery, Custom3:SideSwitch_5_Legs, symbol Switch:SW_DPDT_x2
- D2: footprint (none) -> Diode_SMD:D_SOD-323
- J10: footprint (none) -> Connector_PinSocket_2.54mm:PinSocket_1x04_P2.54mm_Vertical
- J11: footprint (none) -> Custom3:Conn_01x02_no_Silk
- J12: footprint (none) -> Connector_PinSocket_2.54mm:PinSocket_1x07_P2.54mm_Vertical
- J15, J2, J6: footprint Connector_PinHeader_2.54mm:PinHeader_1x02_P2.54mm_Vertical -> Custom3:Conn_01x02_no_Silk
- R10, R11, R12, R15, R16, R17, R18, R19, R20, R21, R22: footprint (none) -> Resistor_SMD:R_0402_1005Metric
- U7: footprint easyeda2kicad:SOT-89-5_L4.5-W2.5-P1.50-LS4.5-TL -> Package_TO_SOT_SMD:SOT-89-5
Connections:
- net +5V is gone; now on net VSYS: J2.1 (Pin_1)
- net BCLK is gone; now on net AUDIO_BCLK: J12.2 (Pin_2)
- net DIN is gone; now on net AUDIO_DIN: J12.3 (Pin_3)
- net LRC is gone; now on net AUDIO_LRC: J12.1 (Pin_1)
- net +3.3V: now also U6.1 (VCC); no longer J12.7 (Pin_7), U6.2 (VCC)
- net GND: now also U6.2 (GND), C2.2, Q4.2 (S); no longer U6.1 (GND), U7.2 (GND)
- net JOYSTICK_LEFT_BTN: now also U3.10 (GPIO17/U1TXD/ADC2_CH6)
- net JOYSTICK_LEFT_HORI: now also U3.12 (GPIO8/TOUCH8/ADC1_CH7/SUBSPICS1)
- net JOYSTICK_LEFT_VERT: now also U3.11 (GPIO18/U1RXD/ADC2_CH7/CLK_OUT3)
- net JOYSTICK_RIGHT_BTN: now also U3.24 (GPIO47/SPICLK_P/SUBSPICLK_P_DIFF)
- net JOYSTICK_RIGHT_HORI: now also U3.22 (GPIO14/TOUCH14/ADC2_CH3/FSPIWP/FSPIDQS/SUBSPIWP)
- net JOYSTICK_RIGHT_VERT: now also U3.23 (GPIO21)
- net LED_BLUE: now also U3.39 (GPIO1/TOUCH1/ADC1_CH0)
- net LED_RED: now also U3.38 (GPIO2/TOUCH2/ADC1_CH1)
- net NRF_CE: now also U6.4 (CE); no longer U6.3 (CE)
- net NRF_CSN: now also U6.3 (~{CSN}); no longer U6.4 (~{CSN})
- net NRF_IRQ: now also U6.7 (IRQ); no longer U6.8 (IRQ)
- net NRF_MISO: now also U6.8 (MISO); no longer U6.7 (MISO)
- net NRF_MOSI: now also U6.5 (MOSI); no longer U6.6 (MOSI)
- net NRF_SCK: now also U6.6 (SCK); no longer U6.5 (SCK)
- net VBAT: now also SW5.3 (C); no longer J4.1 (Pin_1)
- net VSYS: now also J12.7 (Pin_7), C2.1
- net at R11.1, R12.2: now also Q4.1 (G)
- net at D2.2 (A), J11.2 (Pin_2): now also Q4.3 (D)
- net AUDIO_LRC: now reaches U3.28 (SPIIO6/GPIO35/FSPID/SUBSPID)
- net AUDIO_BCLK: now reaches U3.29 (SPIIO7/GPIO36/FSPICLK/SUBSPICLK)
- net AUDIO_DIN: now reaches U3.30 (SPIDQS/GPIO37/FSPIQ/SUBSPIQ)
- net GAIN: no longer names the net of J12.4 (Pin_4)
- net SD: no longer names the net of J12.5 (Pin_5)
- new net: J4.1 (Pin_1), SW5.2 (B)
- no-connect marks 3 -> 7
Other:
- note removed: "These connectors are for connecting external 5V boost module"
- moved on the sheet: D3, D4, H1, H2, H3, H4, J12, J4, J5, R13, R14, U7

Commit message: Transmitter PCB almost done in kicad
Parts:
- removed J10: OLED, Connector_PinSocket_2.54mm:PinSocket_1x04_P2.54mm_Vertical, symbol Connector_Generic:Conn_01x04
- added R23, R24, R25: 10k, Resistor_SMD:R_0402_1005Metric, symbol Device:R_Small
- added SW6, SW7: KAN0641-0431B-L, easyeda2kicad:KEY-SMD_4P-L6.0-W6.0-P4.50-LS10.0, symbol easyeda2kicad:KAN0641-0431B-L
Connections:
- net +3.3V: now also R23.1, R24.1, R25.1
- net AUX_SWITCH_1: now also U3.12 (GPIO8/TOUCH8/ADC1_CH7/SUBSPICS1)
- net AUX_SWITCH_2: now also U3.39 (GPIO1/TOUCH1/ADC1_CH0)
- net BATT_VOLTAGE: now also U3.22 (GPIO14/TOUCH14/ADC2_CH3/FSPIWP/FSPIDQS/SUBSPIWP)
- net DISPLAY_TFT_A0: now also U3.9 (GPIO16/U0CTS/ADC2_CH5/XTAL_32K_N)
- net DISPLAY_TFT_CS: now also U3.7 (GPIO7/TOUCH7/ADC1_CH6)
- net DISPLAY_TFT_RESET: now also U3.8 (GPIO15/U0RTS/ADC2_CH4/XTAL_32K_P)
- net DISPLAY_TFT_SCK: now also U3.11 (GPIO18/U1RXD/ADC2_CH7/CLK_OUT3)
- net DISPLAY_TFT_SDA: now also U3.10 (GPIO17/U1TXD/ADC2_CH6)
- net GND: now also SW6.3, SW6.4, SW7.3, SW7.4
- net JOYSTICK_LEFT_BTN: now also U3.15 (GPIO3/TOUCH3/ADC1_CH2); no longer U3.10 (GPIO17/U1TXD/ADC2_CH6)
- net JOYSTICK_LEFT_HORI: now also U3.18 (GPIO10/TOUCH10/ADC1_CH9/FSPICS0/FSPIIO4/SUBSPICS0); no longer U3.12 (GPIO8/TOUCH8/ADC1_CH7/SUBSPICS1)
- net JOYSTICK_LEFT_VERT: now also U3.17 (GPIO9/TOUCH9/ADC1_CH8/FSPIHD/SUBSPIHD); no longer U3.11 (GPIO18/U1RXD/ADC2_CH7/CLK_OUT3)
- net JOYSTICK_RIGHT_BTN: now also U3.21 (GPIO13/TOUCH13/ADC2_CH2/FSPIQ/FSPIIO7/SUBSPIQ); no longer U3.24 (GPIO47/SPICLK_P/SUBSPICLK_P_DIFF)
- net JOYSTICK_RIGHT_HORI: now also U3.19 (GPIO11/TOUCH11/ADC2_CH0/FSPID/FSPIIO5/SUBSPID); no longer U3.22 (GPIO14/TOUCH14/ADC2_CH3/FSPIWP/FSPIDQS/SUBSPIWP)
- net JOYSTICK_RIGHT_VERT: now also U3.20 (GPIO12/TOUCH12/ADC2_CH1/FSPICLK/FSPIIO6/SUBSPICLK); no longer U3.23 (GPIO21)
- net LED_BLUE: now also U3.16 (GPIO46); no longer U3.39 (GPIO1/TOUCH1/ADC1_CH0)
- net NRF_CE: now also U3.5 (GPIO5/TOUCH5/ADC1_CH4)
- net NRF_CSN: now also U3.6 (GPIO6/TOUCH6/ADC1_CH5)
- net NRF_IRQ: now also U3.33 (MTDO/GPIO40/CLK_OUT2)
- net NRF_MISO: now also U3.35 (MTMS/GPIO42)
- net NRF_MOSI: now also U3.34 (MTDI/GPIO41/CLK_OUT1)
- net NRF_SCK: now also U3.4 (GPIO4/TOUCH4/ADC1_CH3)
- net USB_SENSE: now also U3.24 (GPIO47/SPICLK_P/SUBSPICLK_P_DIFF)
- net VIBRATION_MOTOR: now also U3.25 (GPIO48/SPICLK_N/SUBSPICLK_N_DIFF)
- net ~{CHRG}: now also U3.23 (GPIO21)
- net BTN_RIGHT: now reaches U3.31 (GPIO38/FSPIWP/SUBSPIWP)
- net BTN_RIGHT: now also R25.2, SW7.1, SW7.2
- net BTN_LEFT: now reaches U3.32 (MTCK/GPIO39/CLK_OUT3/SUBSPICS1)
- net BTN_LEFT: now also R24.2, SW6.1, SW6.2
- net DISPLAY_TFT_LED: no longer names the net of J9.1 (Pin_1)
- net DISPLAY_TFT_LED: now also R23.2
- no-connect marks 7 -> 6
Other:
- moved on the sheet: C15, R15, R16, R17, R18, R19, R20, SW1, SW2, SW3A, SW4A, U6

Commit message: Ordered PCBs for rev A
Parts:
- H1, H2, H3, H4: footprint (none) -> MountingHole:MountingHole_3.2mm_M3_Pad_Via
Connections:
- no-connect marks 6 -> 7
Other:
- note added: "TFT SPI Display"
- note removed: "Displays"
- company: (none) -> Victor Krook
- title: (none) -> asactx
- moved on the sheet: C1, C4, C5, H1, H2, H3, H4, J15, J2, J4, J5, J6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
